File: hardware/PCB_Deckenleuchte/PCB_Deckenleuchte.kicad_pcb (KiCad board)
At the start: 2 copper layers, 1 part, among them U1 IRM-20-3.3

Commit message: Add files via upload
Parts:
- added Bewegungssensor-U1: Conn_01x05_Socket, Connector_JST:JST_XH_B5B-XH-A_1x05_P2.50mm_Vertical, F.Cu at (70.3, 88.8)
- added Bewegungssensor1-U1: Conn_01x05_Socket, Connector_JST:JST_XH_B5B-XH-A_1x05_P2.50mm_Vertical, F.Cu at (70.3, 96.6)
- added Bewegungssensor2-U2: Conn_01x05_Socket, Connector_JST:JST_XH_B5B-XH-A_1x05_P2.50mm_Vertical, F.Cu at (70.3, 104.4)
- added Bewegungssensor3-U2: Conn_01x05_Socket, Connector_JST:JST_XH_B5B-XH-A_1x05_P2.50mm_Vertical, F.Cu at (70.3, 112.2)
- added Helligkeitsensor1: Conn_01x05_Socket, Connector_JST:JST_XH_B5B-XH-A_1x05_P2.50mm_Vertical, F.Cu at (70.3, 120.0)
- added Helligkeitsensor2: Conn_01x05_Socket, Connector_JST:JST_XH_B5B-XH-A_1x05_P2.50mm_Vertical, F.Cu at (133.8, 55.2)
- added J1: DFRobot, Connector_JST:JST_PH_B4B-PH-K_1x04_P2.00mm_Vertical, F.Cu at (72.0, 130.6)
- added PS1: IRM-30-5, IRM-30-5:CONV_IRM-30-5, F.Cu at (218.8, 40.5)
- added PS2: ~, third_party_components:DC5-36-TO-DC3V3-5, F.Cu at (39.2, 167.2)
- added U2: DEVKIT_V1_ESP32-WROOM-32_Slave, DEVKIT_V1_ESP32-WROOM-32:MODULE_DEVKIT_V1_ESP32-WROOM-32, F.Cu at (51.9, 111.7)
- U1: value IRM-20-3.3 -> DEVKIT_V1_ESP32-WROOM-32_Master; footprint Converter_ACDC:Converter_ACDC_MeanWell_IRM-20-xx_THT -> DEVKIT_V1_ESP32-WROOM-32:MODULE_DEVKIT_V1_ESP32-WROOM-32
- moved U1 86.4 mm to (120.4, 113.1), turned to 180 degrees
Connections:
- U1 pad 2: unconnected-(U1-AC/N-Pad2) -> GND
